File: Delay No More/delaynomore.kicad_pcb (KiCad board)
At the start: 2 copper layers, 40.3 x 128.5 mm, 10 parts

Commit message: Add files via upload
Parts:
- removed the REF** at (30.0, 56.5)
- removed the TP1 at (5.00, 82.0)
- removed the TP1 at (35.0, 82.0)
- removed the TP1 at (25.0, 82.0)
- removed the TP1 at (15.0, 82.0)
- removed the TP1 at (25.0, 97.5)
- added REF**: 5mm_mounting_hole_LED, custom footprints:5mm_mounting_hole_LED, F.Cu at (20.2, 70.5)
- moved TP1 5.20 mm to (20.2, 97.5)
- moved TP1 2.70 mm to (7.70, 97.5)
- moved TP1 1.80 mm to (33.2, 97.5)
- moved REF** 0.35 mm to (20.2, 123.8)
Other:
- outline, holes or cut-outs redrawn
- board text added: "C V"
- board text added: "COARSE"
- board text added: "DELAY B"
- board text added: "Delay No More"
- board text added: "FINE"
- board text added: "IN"
- board text added: "WET/DRY"
- board text added: "fbA"
- board text added: "fbB"
- board text added: "fbB>A"
- board text added: "ffA>B"
- board text removed: "/16"
- board text removed: "/2"
- board text removed: "/4"
- board text removed: "/8"
- board text removed: "DIVINE CMOS"
- board text removed: "IN1"
- board text removed: "IN2"
- board text removed: "SLEW"
- board text removed: "SLEW OUT"
