File: Divide By N/dividebyn.kicad_pcb (KiCad board)
At the start: 2 copper layers, 40.2 x 128.5 mm, 28 parts

Commit message: Add files via upload
Parts:
- removed the REF** at (20.5, 222.0)
- added REF**: potleaf_small_copper, custom footprints:potleaf_small_copper, F.Cu at (20.2, 223.5)
Routing:
- removed copper zone on F.Cu, net GND
