File: Feague/feague.kicad_pcb (KiCad board)
At the start: 2 copper layers, 50.5 x 128.5 mm, 14 parts

Commit message: Add files via upload
Parts:
- removed the REF** at (125.0, 151.0)
- added REF**: potleaf_small_copper, custom footprints:potleaf_small_copper, F.Cu at (125.2, 153.5)
Routing:
- removed copper zone on F.Cu, net GND
