File: Hyperchaos Deluxe/hyperchaosdeluxe.kicad_pcb (KiCad board)
At the start: 2 copper layers, 50.4 x 128.5 mm, 23 parts

Commit message: Add files via upload
Parts:
- removed the REF** at (25.5, 372.5)
- added REF**: potleaf_small_copper, custom footprints:potleaf_small_copper, F.Cu at (25.2, 373.5)
Routing:
- removed copper zone on F.Cu, net GND
