File: ICBINAVCO/icbina.kicad_pcb (KiCad board)
At the start: 2 copper layers, 40.3 x 128.5 mm, 9 parts

Commit message: Add files via upload
Parts:
- removed the REF** at (120.8, 151.5)
- added REF**: potleaf_small_copper, custom footprints:potleaf_small_copper, F.Cu at (120.0, 153.4)
Routing:
- removed copper zone on F.Cu, net GND
