File: Kareishuu VCO/kareishuuvco.kicad_pcb (KiCad board)
At the start: 2 copper layers, 50.5 x 128.5 mm, 10 parts

Commit message: Add files via upload
Parts:
- removed the REF** at (25.0, 121.0)
- added REF**: potleaf_small_copper, custom footprints:potleaf_small_copper, F.Cu at (25.2, 123.6)
Routing:
- removed copper zone on F.Cu, net GND
