File: Sauce of Unce/sauceofunce.kicad_pcb (KiCad board)
At the start: 2 copper layers, 50.4 x 128.5 mm, 10 parts

Commit message: Add files via upload
Parts:
- removed the REF** at (125.8, 20.2)
- added REF**: potleaf_small_copper, custom footprints:potleaf_small_copper, F.Cu at (125.0, 23.2)
Routing:
- removed copper zone on F.Cu, net GND
