File: Sloths/sloths.kicad_pcb (KiCad board)
At the start: 2 copper layers, 40.3 x 128.5 mm, 17 parts

Commit message: Add files via upload
Parts:
- removed the REF** at (20.8, 121.5)
- added REF**: potleaf_small_copper, custom footprints:potleaf_small_copper, F.Cu at (20.6, 123.5)
Routing:
- removed copper zone on F.Cu, net GND
