File: Sly Grogan/slygrogan.kicad_pcb (KiCad board)
At the start: 2 copper layers, 40.3 x 128.5 mm, 10 parts

Commit message: Add files via upload
Parts:
- removed the REF** at (20.8, 121.5)
- added REF**: potleaf_small_copper, custom footprints:potleaf_small_copper, F.Cu at (20.0, 123.7)
Routing:
- removed copper zone on F.Cu, net GND
