File: Tracky Dacks/trackydacks.kicad_pcb (KiCad board)
At the start: 2 copper layers, 40.2 x 128.5 mm, 9 parts

Commit message: Add files via upload
Parts:
- removed the REF** at (120.5, 20.8)
- added REF**: potleaf_small_copper, custom footprints:potleaf_small_copper, F.Cu at (120.0, 23.7)
Routing:
- removed copper zone on F.Cu, net GND
