File: Helvetica Scenario/helveticascenario.kicad_pcb (KiCad board)
At the start: 2 copper layers, 40.2 x 128.5 mm, 13 parts

Commit message: Add files via upload
Parts:
- removed the REF** at (20.5, 371.5)
- added REF**: potleaf_small_copper, custom footprints:potleaf_small_copper, F.Cu at (20.2, 373.8)
Routing:
- removed copper zone on F.Cu, net GND

Commit message: Add files via upload
Parts:
- added REF**: 3mm_mounting_hole_LED, custom footprints:3mm_mounting_hole_LED, F.Cu at (5.00, 306.5)
- added REF**: 3mm_mounting_hole_LED, custom footprints:3mm_mounting_hole_LED, F.Cu at (25.0, 306.5)
