File: Hypster/hypster.kicad_pcb (KiCad board)
At the start: 2 copper layers, 60.5 x 128.5 mm, 18 parts

Commit message: Add files via upload
Parts:
- removed the REF** at (30.8, 371.2)
- added REF**: potleaf_small_copper, custom footprints:potleaf_small_copper, F.Cu at (30.0, 373.8)
Routing:
- removed copper zone on F.Cu, net GND

Commit message: Add files via upload
Parts:
- removed the TP1 at (10.2, 324.2)
- removed the TP1 at (50.2, 324.2)
- added REF**: 6.35mm_mounting_hole_miniswitch, custom footprints:6.35mm_mounting_hole_miniswitch, F.Cu at (10.2, 324.2)
- added REF**: 6.35mm_mounting_hole_miniswitch, custom footprints:6.35mm_mounting_hole_miniswitch, F.Cu at (50.2, 324.2)
Changed lines of the file:
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@@
   (page A4)
   (layers
-    (0 F.Cu signal)
-    (31 B.Cu signal)
+    (0 F.Cu signal hide)
+    (31 B.Cu signal hide)
     (32 B.Adhes user)
     (33 F.Adhes user)
@@
     (mod_text_size 1 1)
     (mod_text_width 0.15)
-    (pad_size 1.524 1.524)
-    (pad_drill 0.762)
+    (pad_size 6.4 6.4)
+    (pad_drill 6.35)
     (pad_to_mask_clearance 0.051)
     (solder_mask_min_width 0.25)
@@
     (uvia_drill 0.1)
     (add_net GND)
+  )
+  (module "custom footprints:6.35mm_mounting_hole_miniswitch" (layer F.Cu)
+    (at 10.25 324.25)
+    (descr "Through hole straight socket strip, 1x01, 2.54mm pitch, single row (from Kicad 4.0.7), script generated")
+    (tags "Through hole socket strip THT 1x01 2.54mm single row")
+    (fp_text reference REF** (at 0 -2.77) (layer F.SilkS) hide
+      (effects (font (size 1 1) (thickness 0.15)))
+    )
+    (fp_text value 6.35mm_mounting_hole_miniswitch (at 0 2.77) (layer F.Fab)
+      (effects (font (size 1 1) (thickness 0.15)))
+    )
+    (pad 1 thru_hole circle (at 0 0) (size 6.4 6.4) (drill 6.35) (layers *.Cu *.Mask)
+      (net 1 GND))
+    (model ${KISYS3DMOD}/Connector_PinSocket_2.54mm.3dshapes/PinSocket_1x01_P2.54mm_Vertical.wrl
+      (at (xyz 0 0 0))
+      (scale (xyz 1 1 1))
+      (rotate (xyz 0 0 0))
+    )
+  )
+  (module "custom footprints:6.35mm_mounting_hole_miniswitch" (layer F.Cu)
+    (at 50.25 324.25)
+    (descr "Through hole straight socket strip, 1x01, 2.54mm pitch, single row (from Kicad 4.0.7), script generated")
+    (tags "Through hole socket strip THT 1x01 2.54mm single row")
+    (fp_text reference REF** (at 0 -2.77) (layer F.SilkS) hide
+      (effects (font (size 1 1) (thickness 0.15)))
+    )
+    (fp_text value 6.35mm_mounting_hole_miniswitch (at 0 2.77) (layer F.Fab)
+      (effects (font (size 1 1) (thickness 0.15)))
+    )
+    (pad 1 thru_hole circle (at 0 0) (size 6.4 6.4) (drill 6.35) (layers *.Cu *.Mask)
+      (net 1 GND))
+    (model ${KISYS3DMOD}/Connector_PinSocket_2.54mm.3dshapes/PinSocket_1x01_P2.54mm_Vertical.wrl
+      (at (xyz 0 0 0))
+      (scale (xyz 1 1 1))
+      (rotate (xyz 0 0 0))
+    )
   )
   (module "custom footprints:potleaf_small_copper" (layer F.Cu)
@@
     (fp_line (start -0.5588 -2.4892) (end -0.54484 -2.202223) (layer F.Mask) (width 0.000002))
   )
-  (module "custom footprints:6mm_mounting_hole_thonkiconn" (layer F.Cu)
-    (at 10.25 324.25)
-    (descr "Through hole straight socket strip, 1x01, 2.54mm pitch, single row (from Kicad 4.0.7), script generated")
-    (tags "Through hole socket strip THT 1x01 2.54mm single row")
-    (fp_text reference TP1 (at 0 -2.77) (layer F.SilkS) hide
-      (effects (font (size 1 1) (thickness 0.15)))
-    )
-    (fp_text value TestPoint (at 0 2.77) (layer F.Fab)
-      (effects (font (size 1 1) (thickness 0.15)))
-    )
-    (pad 1 thru_hole circle (at 0 0) (size 6.1 6.1) (drill 6) (layers *.Cu *.Mask)
-      (net 1 GND))
-    (model ${KISYS3DMOD}/Connector_PinSocket_2.54mm.3dshapes/PinSocket_1x01_P2.54mm_Vertical.wrl
-      (at (xyz 0 0 0))
-      (scale (xyz 1 1 1))
-      (rotate (xyz 0 0 0))
-    )
-  )
-  (module "custom footprints:6mm_mounting_hole_thonkiconn" (layer F.Cu)
-    (at 50.25 324.25)
-    (descr "Through hole straight socket strip, 1x01, 2.54mm pitch, single row (from Kicad 4.0.7), script generated")
-    (tags "Through hole socket strip THT 1x01 2.54mm single row")
-    (fp_text reference TP1 (at 0 -2.77) (layer F.SilkS) hide
-      (effects (font (size 1 1) (thickness 0.15)))
-    )
-    (fp_text value TestPoint (at 0 2.77) (layer F.Fab)
-      (effects (font (size 1 1) (thickness 0.15)))
-    )
-    (pad 1 thru_hole circle (at 0 0) (size 6.1 6.1) (drill 6) (layers *.Cu *.Mask)
-      (net 1 GND))
-    (model ${KISYS3DMOD}/Connector_PinSocket_2.54mm.3dshapes/PinSocket_1x01_P2.54mm_Vertical.wrl
-      (at (xyz 0 0 0))
-      (scale (xyz 1 1 1))
-      (rotate (xyz 0 0 0))
-    )
-  )
   (module "custom footprints:5mm_mounting_hole_LED" (layer F.Cu)
